File: pcb/macro-pad.kicad_sch (KiCad schematic)
At the start: 5 parts, among them J1 Conn_01x04_Pin

Commit message: Add files via upload
Parts:
- removed RZ1: RP2040-Zero, modfile:RP2040-Zero, symbol rp2040-zero:RP2040-Zero
- added D1, D2, D5, D6: SK6812MINI-E, LED_SMD:LED_SK6812MINI-E_3.2x2.8mm_P1.5mm_ReverseMount, symbol LED:SK6812MINI-E
- added D10, D11, D12, D13, D14, D15, D7, D8, D9: 1N4148, Diode_THT:D_DO-35_SOD27_P7.62mm_Horizontal, symbol Diode:1N4148
- added H1, H3, H4: MountingHole, MountingHole:MountingHole_3.2mm_M3, symbol Mechanical:MountingHole
- added MX4: 1,0, marbastlib-xp-mx:SW_MX_Reversible_1u, symbol marbastlib-mx:MX_SW_HS_CPG151101S11
- added MX5: 1,1, marbastlib-xp-mx:SW_MX_Reversible_1u, symbol marbastlib-mx:MX_SW_HS_CPG151101S11
- added MX6: 1,2, marbastlib-xp-mx:SW_MX_Reversible_1u, symbol marbastlib-mx:MX_SW_HS_CPG151101S11
- added MX7: 2,0, marbastlib-xp-mx:SW_MX_Reversible_1u, symbol marbastlib-mx:MX_SW_HS_CPG151101S11
- added MX8: 2,1, marbastlib-xp-mx:SW_MX_Reversible_1u, symbol marbastlib-mx:MX_SW_HS_CPG151101S11
- added MX9: 2,2, marbastlib-xp-mx:SW_MX_Reversible_1u, symbol marbastlib-mx:MX_SW_HS_CPG151101S11
- added SW1: RotaryEncoder_Switch_MP, Rotary_Encoder:RotaryEncoder_Alps_EC11E-Switch_Vertical_H20mm_CircularMountingHoles, symbol Device:RotaryEncoder_Switch_MP
- added U1: XIAO-RP2040-SMD, Seeed_Studio_XIAO_Series:XIAO-RP2040-SMD, symbol Seeed_Studio_XIAO_Series:XIAO-RP2040-SMD
- MX1: value MX_SW_HS -> 0,0; footprint marbastlib-mx:SW_MX_HS_CPG151101S11_1u -> marbastlib-xp-mx:SW_MX_Reversible_1u
- MX2: value MX_SW_HS -> 0,1; footprint marbastlib-mx:SW_MX_HS_CPG151101S11_1u -> marbastlib-xp-mx:SW_MX_Reversible_1u
- MX3: value MX_SW_HS -> 0,2; footprint marbastlib-mx:SW_MX_HS_CPG151101S11_1u -> marbastlib-xp-mx:SW_MX_Reversible_1u
Connections:
- net - is gone; now on net Column 0: MX3.1
- net MUTE is gone; now on net Column 0: MX2.1
- net GND: now also D1.1 (VSS), D2.1 (VSS), D5.1 (VSS), D6.1 (VSS), SW1.C, SW1.MP, U1.13 (GND); no longer MX1.2, MX2.2, MX3.2
- net SCL: now also U1.6 (D5)
- net SDA: now also U1.5 (D4)
- net + renamed Column 0
- net Column 0: now also U1.1 (D0)
- net VCC renamed 3V3
- net 3V3: now also U1.12 (3V3_OUT)
- new net: D10.2 (A), MX9.2
- new net: D9.2 (A), MX6.2
- new net: D11.2 (A), MX5.2
- new net: D13.2 (A), MX7.2
- new net: D2.4 (DOUT), D6.2 (DIN)
- new net: D5.2 (DIN), D6.4 (DOUT)
- new net: D7.2 (A), MX3.2
- new net: D1.4 (DOUT), D2.2 (DIN)
- new net: D12.2 (A), MX8.2
- new net: D15.2 (A), MX1.2
- new net: D8.2 (A), MX2.2
- new net: D14.2 (A), MX4.2
- new net 5V: D1.3 (VDD), D2.3 (VDD), D5.3 (VDD), D6.3 (VDD), U1.14 (VBUS)
- new net Column 1: MX4.1, MX5.1, MX6.1, U1.2 (D1)
- new net Column 2: MX7.1, MX8.1, MX9.1, U1.3 (D2)
- new net LED INPUT: D1.2 (DIN), U1.8 (D7)
- new net Row 0: D13.1 (K), D14.1 (K), D15.1 (K), U1.4 (D3)
- new net Row 1: D11.1 (K), D12.1 (K), D8.1 (K), U1.7 (D6)
- new net Row 2: D10.1 (K), D7.1 (K), D9.1 (K), U1.11 (D10)
- new net Signal 1: SW1.A, U1.10 (D9)
- new net Signal 2: SW1.B, U1.9 (D8)
